File: Hardware/ecu-pcb/apps.kicad_sch (KiCad schematic)
At the start: 12 parts, among them U9 LM358DR2G

Commit message: Updated Schematic
Other:
- title: (none) -> Apps 
Changed lines of the file:
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@@
 (kicad_sch (version 20211123) (generator eeschema)
   (paper "A4")
+  (title_block
+    (title "Apps ")
+  )
   (junction (at 148.59 66.675) (diameter 0) (color 0 0 0 0)
   )
