File: Hardware/ecu-pcb/gpio.kicad_sch (KiCad schematic)
At the start: 7 parts, among them CN7 B2B-XH-A(LF)(SN), Q5 AO3400A

Commit message: Updated Schematic
Parts:
- renumbered R26 to R36
Changed lines of the file:
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@@
   (symbol (lib_id "power:GND") (at 154.94 101.6 0) (unit 1)
     (in_bom yes) (on_board yes) (fields_autoplaced)
-    (property "Reference" "#PWR0191" (id 0) (at 154.94 107.95 0)
+    (property "Reference" "#PWR0217" (id 0) (at 154.94 107.95 0)
       (effects (font (size 1.27 1.27)) hide)
     )
@@
   (symbol (lib_id "easyeda2kicad:1kΩ 0402 50V") (at 154.94 86.36 90) (unit 1)
     (in_bom yes) (on_board yes) (fields_autoplaced)
-    (property "Reference" "R26" (id 0) (at 156.718 85.0899 90)
+    (property "Reference" "R36" (id 0) (at 156.718 85.0899 90)
       (effects (font (size 1.27 1.27)) (justify right))
     )
