File: Hardware/ecu-pcb/iso.kicad_sch (KiCad schematic)
At the start: 12 parts

Commit message: Updated Schematic
Parts:
- gave numbers to parts that had none: 11
- renumbered R22 to R32
Other:
- title: (none) -> Apps Measurement Unit
Changed lines of the file:
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@@
 (kicad_sch (version 20211123) (generator eeschema)
   (paper "A4")
+  (title_block
+    (title "Apps Measurement Unit")
+  )
   (junction (at 214.122 50.8) (diameter 0) (color 0 0 0 0)
   )
@@
   (symbol (lib_id "easyeda2kicad:600Ω 200mA") (at 122.428 32.512 0) (unit 1)
     (in_bom yes) (on_board yes) (fields_autoplaced)
-    (property "Reference" "L?" (id 0) (at 122.428 26.67 0))
+    (property "Reference" "L15" (id 0) (at 122.428 26.67 0))
     (property "Value" "600Ω 200mA" (id 1) (at 122.428 29.21 0))
     (property "Footprint" "easyeda2kicad:L0603" (id 2) (at 122.428 40.132 0)
@@
   (symbol (lib_id "power:GND") (at 221.742 81.28 0) (unit 1)
     (in_bom yes) (on_board yes) (fields_autoplaced)
-    (property "Reference" "#PWR?" (id 0) (at 221.742 87.63 0)
+    (property "Reference" "#PWR0203" (id 0) (at 221.742 87.63 0)
       (effects (font (size 1.27 1.27)) hide)
     )
@@
   (symbol (lib_id "easyeda2kicad:1kΩ 0402 50V") (at 240.03 46.736 90) (unit 1)
     (in_bom yes) (on_board yes) (fields_autoplaced)
-    (property "Reference" "R?" (id 0) (at 242.57 45.4659 90)
+    (property "Reference" "R33" (id 0) (at 242.57 45.4659 90)
       (effects (font (size 1.27 1.27)) (justify right))
     )
@@
   (symbol (lib_id "easyeda2kicad:25V 10uF X5R ±10% 0805") (at 117.348 36.322 90) (unit 1)
     (in_bom yes) (on_board yes)
-    (property "Reference" "C?" (id 0) (at 118.364 34.798 90)
+    (property "Reference" "C49" (id 0) (at 118.364 34.798 90)
       (effects (font (size 1.27 1.27)) (justify right))
     )
@@
   (symbol (lib_id "easyeda2kicad:25V 1uF X5R ±10% 0402") (at 86.868 42.672 90) (unit 1)
     (in_bom yes) (on_board yes)
-    (property "Reference" "C?" (id 0) (at 79.756 42.672 90)
+    (property "Reference" "C53" (id 0) (at 79.756 42.672 90)
       (effects (font (size 1.27 1.27)) (justify right))
     )
@@
   (symbol (lib_id "easyeda2kicad:25V 1uF X5R ±10% 0402") (at 141.986 37.592 90) (unit 1)
     (in_bom yes) (on_board yes) (fields_autoplaced)
-    (property "Reference" "C?" (id 0) (at 144.78 36.3219 90)
+    (property "Reference" "C51" (id 0) (at 144.78 36.3219 90)
       (effects (font (size 1.27 1.27)) (justify right))
     )
@@
   (symbol (lib_id "easyeda2kicad:B3B-PH-K-S(LF)(SN)") (at 246.38 36.576 180) (unit 1)
     (in_bom yes) (on_board yes) (fields_autoplaced)
-    (property "Reference" "CN?" (id 0) (at 254.508 35.3059 0)
+    (property "Reference" "CN6" (id 0) (at 254.508 35.3059 0)
       (effects (font (size 1.27 1.27)) (justify right))
     )
@@
   (symbol (lib_id "easyeda2kicad:HT7550-1_C16106") (at 107.188 37.592 0) (unit 1)
     (in_bom yes) (on_board yes) (fields_autoplaced)
-    (property "Reference" "U?" (id 0) (at 107.188 25.4 0))
+    (property "Reference" "U10" (id 0) (at 107.188 25.4 0))
     (property "Value" "HT7550" (id 1) (at 107.188 27.94 0))
     (property "Footprint" "easyeda2kicad:SOT-89-3_L4.5-W2.5-P1.50-LS4.2-BR" (id 2) (at 107.188 50.292 0)
@@
   (symbol (lib_id "easyeda2kicad:25V 1uF X5R ±10% 0402") (at 127.508 37.592 90) (unit 1)
     (in_bom yes) (on_board yes) (fields_autoplaced)
-    (property "Reference" "C?" (id 0) (at 130.302 36.3219 90)
+    (property "Reference" "C50" (id 0) (at 130.302 36.3219 90)
       (effects (font (size 1.27 1.27)) (justify right))
     )
@@
   (symbol (lib_id "easyeda2kicad:600Ω 200mA") (at 91.948 37.592 0) (unit 1)
     (in_bom yes) (on_board yes) (fields_autoplaced)
-    (property "Reference" "L?" (id 0) (at 91.948 31.75 0))
+    (property "Reference" "L16" (id 0) (at 91.948 31.75 0))
     (property "Value" "600Ω 200mA" (id 1) (at 91.948 34.29 0))
     (property "Footprint" "easyeda2kicad:L0603" (id 2) (at 91.948 45.212 0)
@@
   (symbol (lib_id "easyeda2kicad:25V 10uF X5R ±10% 0805") (at 97.028 41.402 90) (unit 1)
     (in_bom yes) (on_board yes)
-    (property "Reference" "C?" (id 0) (at 98.044 39.878 90)
+    (property "Reference" "C52" (id 0) (at 98.044 39.878 90)
       (effects (font (size 1.27 1.27)) (justify right))
     )
@@
   (symbol (lib_id "power:GND") (at 97.028 45.212 0) (unit 1)
     (in_bom yes) (on_board yes) (fields_autoplaced)
-    (property "Reference" "#PWR?" (id 0) (at 97.028 51.562 0)
+    (property "Reference" "#PWR0208" (id 0) (at 97.028 51.562 0)
       (effects (font (size 1.27 1.27)) hide)
     )
@@
   (symbol (lib_id "power:GND") (at 127.508 42.672 0) (unit 1)
     (in_bom yes) (on_board yes) (fields_autoplaced)
-    (property "Reference" "#PWR?" (id 0) (at 127.508 49.022 0)
+    (property "Reference" "#PWR0206" (id 0) (at 127.508 49.022 0)
       (effects (font (size 1.27 1.27)) hide)
     )
@@
   (symbol (lib_id "power:GND") (at 86.868 47.752 0) (unit 1)
     (in_bom yes) (on_board yes) (fields_autoplaced)
-    (property "Reference" "#PWR?" (id 0) (at 86.868 54.102 0)
+    (property "Reference" "#PWR0209" (id 0) (at 86.868 54.102 0)
       (effects (font (size 1.27 1.27)) hide)
     )
@@
   (symbol (lib_id "easyeda2kicad:100Ω 0402 50V") (at 234.95 36.576 0) (unit 1)
     (in_bom yes) (on_board yes)
-    (property "Reference" "R22" (id 0) (at 231.14 38.862 0))
+    (property "Reference" "R32" (id 0) (at 231.14 38.862 0))
     (property "Value" "100Ω 0402 50V" (id 1) (at 233.934 33.528 0))
     (property "Footprint" "easyeda2kicad:R0402" (id 2) (at 234.95 44.196 0)
@@
   (symbol (lib_id "power:GND") (at 240.03 51.816 0) (unit 1)
     (in_bom yes) (on_board yes) (fields_autoplaced)
-    (property "Reference" "#PWR?" (id 0) (at 240.03 58.166 0)
+    (property "Reference" "#PWR0204" (id 0) (at 240.03 58.166 0)
       (effects (font (size 1.27 1.27)) hide)
     )
@@
   (symbol (lib_id "easyeda2kicad:SMF05CT1G") (at 221.742 66.04 90) (unit 1)
     (in_bom yes) (on_board yes) (fields_autoplaced)
-    (property "Reference" "D?" (id 0) (at 235.712 64.7699 90)
+    (property "Reference" "D10" (id 0) (at 235.712 64.7699 90)
       (effects (font (size 1.27 1.27)) (justify right))
     )
@@
   (symbol (lib_id "power:GND") (at 117.348 42.672 0) (unit 1)
     (in_bom yes) (on_board yes) (fields_autoplaced)
-    (property "Reference" "#PWR?" (id 0) (at 117.348 49.022 0)
+    (property "Reference" "#PWR0211" (id 0) (at 117.348 49.022 0)
       (effects (font (size 1.27 1.27)) hide)
     )
@@
   (symbol (lib_id "power:GND") (at 141.986 42.672 0) (unit 1)
     (in_bom yes) (on_board yes) (fields_autoplaced)
-    (property "Reference" "#PWR?" (id 0) (at 141.986 49.022 0)
-      (effects (font (size 1.27 1.27)) hide)
-    )
+    (property "Reference" "#PWR0205" (id 0) (at 141.986 49.022 0)
+      (effects (font (size 1.27 1.27)) hide)
+    )
