File: Hardware/ecu-pcb/sensor.kicad_sch (KiCad schematic)
At the start: 8 parts, among them CN10 B3B-PH-K-S(LF)(SN)

Commit message: Updated Schematic
Parts:
- JP1: footprint (none) -> Jumper:SolderJumper-3_P1.3mm_Bridged12_Pad1.0x1.5mm_NumberLabels
Changed lines of the file:
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@@
     (property "Reference" "JP1" (id 0) (at 192.024 53.34 0))
     (property "Value" "SolderJumper_3_Bridged12" (id 1) (at 192.024 55.88 0))
-    (property "Footprint" "" (id 2) (at 192.024 59.817 0)
+    (property "Footprint" "Jumper:SolderJumper-3_P1.3mm_Bridged12_Pad1.0x1.5mm_NumberLabels" (id 2) (at 192.024 59.817 0)
       (effects (font (size 1.27 1.27)) hide)
     )
