File: Hardware/ecu-pcb/PAM8303.kicad_sch (KiCad schematic)
At the start: 11 parts, among them U6 PAM8303DBSC

Commit message: Updated Schematic
Other:
- title: (none) -> RTDS Audio Amplifier
Changed lines of the file:
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@@
 (kicad_sch (version 20211123) (generator eeschema)
   (paper "A4")
+  (title_block
+    (title "RTDS Audio Amplifier")
+  )
   (wire (pts (xy 137.668 118.11) (xy 137.668 117.348))
     (stroke (width 0) (type default) (color 0 0 0 0))

Commit message: PCB Done
Connections:
- net Vin: no longer C26.2, C27.2, C28.2, C31.1, L9.2, U6.2 (PVDD), U6.3 (VDD)
- new net Vin_f: C26.2, C27.2, C28.2, C31.1, L9.2, U6.2 (PVDD), U6.3 (VDD)
Changed lines of the file:
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@@
+    (stroke (width 0) (type default) (color 0 0 0 0))
+  )
+  (wire (pts (xy 112.268 114.808) (xy 112.268 112.268))
     (stroke (width 0) (type default) (color 0 0 0 0))
   )
@@
     (stroke (width 0) (type default) (color 0 0 0 0))
   )
-  (wire (pts (xy 112.268 112.268) (xy 112.268 114.808))
-    (stroke (width 0) (type default) (color 0 0 0 0))
-  )
-  (label "Vin" (at 60.198 98.298 180)
+  (label "Vin_f" (at 60.198 98.298 180)
     (effects (font (size 1.27 1.27)) (justify right bottom))
   )
-  (label "Vin" (at 59.944 123.19 180)
+  (label "Vin_f" (at 59.944 123.19 180)
     (effects (font (size 1.27 1.27)) (justify right bottom))
   )
-  (label "Vin" (at 72.644 80.264 0)
+  (label "Vin_f" (at 72.644 80.264 0)
     (effects (font (size 1.27 1.27)) (justify left bottom))
   )
-  (label "Vin" (at 112.268 112.268 180)
+  (label "Vin_f" (at 112.268 114.808 180)
     (effects (font (size 1.27 1.27)) (justify right bottom))
   )
-  (label "Vin" (at 59.944 147.32 180)
+  (label "Vin_f" (at 59.944 147.32 180)
     (effects (font (size 1.27 1.27)) (justify right bottom))
   )
