File: Hardware/ecu-pcb/sn230.kicad_sch (KiCad schematic)
At the start: 10 parts

Commit message: Ecu SCH Ready
Parts:
- gave numbers to parts that had none: 10
Changed lines of the file:
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@@
   (symbol (lib_id "easyeda2kicad:600Ω 200mA") (at 107.188 91.694 0) (unit 1)
     (in_bom yes) (on_board yes) (fields_autoplaced)
-    (property "Reference" "L?" (id 0) (at 107.188 85.344 0))
+    (property "Reference" "L4" (id 0) (at 107.188 85.344 0))
     (property "Value" "600Ω 200mA" (id 1) (at 107.188 87.884 0))
     (property "Footprint" "easyeda2kicad:L0603" (id 2) (at 107.188 99.314 0)
@@
   (symbol (lib_id "easyeda2kicad:0Ω 0402 50V") (at 151.638 89.154 180) (unit 1)
     (in_bom yes) (on_board yes)
-    (property "Reference" "R?" (id 0) (at 152.908 86.614 0))
+    (property "Reference" "R7" (id 0) (at 152.908 86.614 0))
     (property "Value" "0Ω" (id 1) (at 149.86 86.868 0))
     (property "Footprint" "easyeda2kicad:R0402" (id 2) (at 151.638 81.534 0)
@@
   (symbol (lib_id "easyeda2kicad:PSM712-LF-T7") (at 173.736 109.22 270) (unit 1)
     (in_bom yes) (on_board yes) (fields_autoplaced)
-    (property "Reference" "D?" (id 0) (at 181.61 108.3299 90)
+    (property "Reference" "D2" (id 0) (at 181.61 108.3299 90)
       (effects (font (size 1.27 1.27)) (justify left))
     )
@@
   (symbol (lib_id "power:GND") (at 173.736 118.11 0) (unit 1)
     (in_bom yes) (on_board yes) (fields_autoplaced)
-    (property "Reference" "#PWR?" (id 0) (at 173.736 124.46 0)
+    (property "Reference" "#PWR0133" (id 0) (at 173.736 124.46 0)
       (effects (font (size 1.27 1.27)) hide)
     )
@@
   (symbol (lib_id "easyeda2kicad:16V 100nF X7R ±10% 0402") (at 112.268 95.504 90) (unit 1)
     (in_bom yes) (on_board yes) (fields_autoplaced)
-    (property "Reference" "C?" (id 0) (at 115.316 94.2339 90)
+    (property "Reference" "C10" (id 0) (at 115.316 94.2339 90)
       (effects (font (size 1.27 1.27)) (justify right))
     )
@@
   (symbol (lib_id "power:GND") (at 112.268 99.314 0) (unit 1)
     (in_bom yes) (on_board yes) (fields_autoplaced)
-    (property "Reference" "#PWR?" (id 0) (at 112.268 105.664 0)
+    (property "Reference" "#PWR0132" (id 0) (at 112.268 105.664 0)
       (effects (font (size 1.27 1.27)) hide)
     )
@@
   (symbol (lib_id "power:GND") (at 146.558 76.454 180) (unit 1)
     (in_bom yes) (on_board yes) (fields_autoplaced)
-    (property "Reference" "#PWR?" (id 0) (at 146.558 70.104 0)
+    (property "Reference" "#PWR0128" (id 0) (at 146.558 70.104 0)
       (effects (font (size 1.27 1.27)) hide)
     )
@@
   (symbol (lib_id "power:+3.3V") (at 102.108 91.694 90) (unit 1)
     (in_bom yes) (on_board yes) (fields_autoplaced)
-    (property "Reference" "#PWR?" (id 0) (at 105.918 91.694 0)
+    (property "Reference" "#PWR0130" (id 0) (at 105.918 91.694 0)
       (effects (font (size 1.27 1.27)) hide)
     )
@@
   (symbol (lib_id "power:GND") (at 126.238 89.154 270) (unit 1)
     (in_bom yes) (on_board yes) (fields_autoplaced)
-    (property "Reference" "#PWR?" (id 0) (at 119.888 89.154 0)
+    (property "Reference" "#PWR0129" (id 0) (at 119.888 89.154 0)
       (effects (font (size 1.27 1.27)) hide)
     )
@@
   (symbol (lib_id "easyeda2kicad:1kΩ 0402 50V") (at 146.558 81.534 90) (unit 1)
     (in_bom yes) (on_board yes) (fields_autoplaced)
-    (property "Reference" "R?" (id 0) (at 148.59 80.2639 90)
+    (property "Reference" "R6" (id 0) (at 148.59 80.2639 90)
       (effects (font (size 1.27 1.27)) (justify right))
     )
@@
   (symbol (lib_id "power:GND") (at 102.108 101.854 0) (unit 1)
     (in_bom yes) (on_board yes) (fields_autoplaced)
-    (property "Reference" "#PWR?" (id 0) (at 102.108 108.204 0)
+    (property "Reference" "#PWR0131" (id 0) (at 102.108 108.204 0)
       (effects (font (size 1.27 1.27)) hide)
     )
@@
   (symbol (lib_id "easyeda2kicad:25V 1uF X5R ±10% 0402") (at 102.108 96.774 90) (unit 1)
     (in_bom yes) (on_board yes) (fields_autoplaced)
-    (property "Reference" "C?" (id 0) (at 105.156 95.5039 90)
+    (property "Reference" "C11" (id 0) (at 105.156 95.5039 90)
       (effects (font (size 1.27 1.27)) (justify right))
     )
@@
   (symbol (lib_id "easyeda2kicad:120Ω 0402 50V") (at 159.766 90.424 90) (unit 1)
     (in_bom yes) (on_board yes) (fields_autoplaced)
-    (property "Reference" "R?" (id 0) (at 162.56 89.1539 90)
+    (property "Reference" "R8" (id 0) (at 162.56 89.1539 90)
       (effects (font (size 1.27 1.27)) (justify right))
     )
@@
   (symbol (lib_id "easyeda2kicad:B2B-XH-A(LF)(SN)") (at 193.802 90.424 0) (unit 1)
     (in_bom yes) (on_board yes) (fields_autoplaced)
-    (property "Reference" "CN?" (id 0) (at 201.676 89.1539 0)
+    (property "Reference" "CN2" (id 0) (at 201.676 89.1539 0)
       (effects (font (size 1.27 1.27)) (justify left))
     )
@@
   (symbol (lib_id "easyeda2kicad:SN65HVD230DR") (at 136.398 90.424 0) (unit 1)
     (in_bom yes) (on_board yes) (fields_autoplaced)
-    (property "Reference" "U?" (id 0) (at 136.398 78.74 0))
+    (property "Reference" "U4" (id 0) (at 136.398 78.74 0))
     (property "Value" "SN65HVD230DR" (id 1) (at 136.398 81.28 0))
     (property "Footprint" "easyeda2kicad:SOIC-8_L4.9-W3.9-P1.27-LS6.0-BL" (id 2) (at 136.398 101.854 0)
@@
   (symbol (lib_id "easyeda2kicad:0Ω 0402 50V") (at 151.638 91.694 0) (unit 1)
     (in_bom yes) (on_board yes)
-    (property "Reference" "R?" (id 0) (at 150.368 94.234 0))
+    (property "Reference" "R9" (id 0) (at 150.368 94.234 0))
     (property "Value" "0Ω" (id 1) (at 153.416 93.98 0))
     (property "Footprint" "easyeda2kicad:R0402" (id 2) (at 151.638 99.314 0)

Commit message: PCB Done
Parts:
- removed CN2: B2B-XH-A(LF)(SN), easyeda2kicad:CONN-TH_B2B-XH-A-LF-SN, symbol easyeda2kicad:B2B-XH-A(LF)(SN)
- added CN2: B3B-PH-K-S(LF)(SN), easyeda2kicad:CONN-TH_B3B-PH-K-S, symbol easyeda2kicad:B3B-PH-K-S(LF)(SN)
Connections:
- net GND: now also CN2.1
- net at D2.1 (A1), R7.1, R8.2: now also CN2.3
- net at D2.2 (A1), R8.1, R9.2: now also CN2.2
Changed lines of the file:
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@@
+    (stroke (width 0) (type default) (color 0 0 0 0))
+  )
+  (wire (pts (xy 187.452 95.504) (xy 187.452 90.424))
     (stroke (width 0) (type default) (color 0 0 0 0))
   )
@@
     (stroke (width 0) (type default) (color 0 0 0 0))
   )
-  (wire (pts (xy 187.452 85.344) (xy 187.452 89.154))
-    (stroke (width 0) (type default) (color 0 0 0 0))
-  )
   (wire (pts (xy 178.816 100.33) (xy 178.816 85.344))
     (stroke (width 0) (type default) (color 0 0 0 0))
@@
     (stroke (width 0) (type default) (color 0 0 0 0))
   )
-  (wire (pts (xy 187.452 91.694) (xy 187.452 95.504))
+  (wire (pts (xy 187.452 90.424) (xy 189.738 90.424))
     (stroke (width 0) (type default) (color 0 0 0 0))
   )
@@
     (stroke (width 0) (type default) (color 0 0 0 0))
   )
-  (wire (pts (xy 178.816 85.344) (xy 187.452 85.344))
+  (wire (pts (xy 178.816 85.344) (xy 189.738 85.344))
     (stroke (width 0) (type default) (color 0 0 0 0))
   )
@@
     (pin "2")
   )
+  (symbol (lib_id "power:GND") (at 189.738 95.504 0) (unit 1)
+    (in_bom yes) (on_board yes) (fields_autoplaced)
+    (property "Reference" "#PWR0239" (id 0) (at 189.738 101.854 0)
+      (effects (font (size 1.27 1.27)) hide)
+    )
+    (property "Value" "GND" (id 1) (at 189.738 100.584 0))
+    (property "Footprint" "" (id 2) (at 189.738 95.504 0)
+      (effects (font (size 1.27 1.27)) hide)
+    )
+    (property "Datasheet" "" (id 3) (at 189.738 95.504 0)
+      (effects (font (size 1.27 1.27)) hide)
+    )
+    (pin "1")
+  )
   (symbol (lib_id "easyeda2kicad:PSM712-LF-T7") (at 173.736 109.22 270) (unit 1)
     (in_bom yes) (on_board yes) (fields_autoplaced)
@@
     (pin "1")
   )
+  (symbol (lib_id "easyeda2kicad:B3B-PH-K-S(LF)(SN)") (at 196.088 90.424 180) (unit 1)
+    (in_bom yes) (on_board yes) (fields_autoplaced)
+    (property "Reference" "CN2" (id 0) (at 204.216 89.1539 0)
+      (effects (font (size 1.27 1.27)) (justify right))
+    )
+    (property "Value" "B3B-PH-K-S(LF)(SN)" (id 1) (at 204.216 91.6939 0)
+      (effects (font (size 1.27 1.27)) (justify right))
+    )
+    (property "Footprint" "easyeda2kicad:CONN-TH_B3B-PH-K-S" (id 2) (at 196.088 77.724 0)
+      (effects (font (size 1.27 1.27)) hide)
+    )
+    (property "Datasheet" "https://lcsc.com/product-detail/PH-Connectors_JST_B3B-PH-K-S-LF-SN_B3B-PH-K-S-LF-SN_C131339.html" (id 3) (at 196.088 75.184 0)
+      (effects (font (size 1.27 1.27)) hide)
+    )
+    (property "Manufacturer" "JST" (id 4) (at 196.088 72.644 0)
+      (effects (font (size 1.27 1.27)) hide)
+    )
+    (property "LCSC Part" "C131339" (id 5) (at 196.088 70.104 0)
+      (effects (font (size 1.27 1.27)) hide)
+    )
+    (property "JLC Part" "Extended Part" (id 6) (at 196.088 67.564 0)
+      (effects (font (size 1.27 1.27)) hide)
+    )
+    (pin "1")
+    (pin "2")
+    (pin "3")
+  )
   (symbol (lib_id "power:GND") (at 146.558 76.454 180) (unit 1)
     (in_bom yes) (on_board yes) (fields_autoplaced)
@@
       (effects (font (size 1.27 1.27)) hide)
     )
-    (pin "1")
-    (pin "2")
-  )
-  (symbol (lib_id "easyeda2kicad:B2B-XH-A(LF)(SN)") (at 193.802 90.424 0) (unit 1)
-    (in_bom yes) (on_board yes) (fields_autoplaced)
-    (property "Reference" "CN2" (id 0) (at 201.676 89.1539 0)
-      (effects (font (size 1.27 1.27)) (justify left))
-    )
-    (property "Value" "B2B-XH-A(LF)(SN)" (id 1) (at 201.676 91.6939 0)
-      (effects (font (size 1.27 1.27)) (justify left))
-    )
-    (property "Footprint" "easyeda2kicad:CONN-TH_B2B-XH-A-LF-SN" (id 2) (at 193.802 99.314 0)
-      (effects (font (size 1.27 1.27)) hide)
-    )
-    (property "Datasheet" "https://lcsc.com/product-detail/XH-Connectors_JST_B2B-XH-A-LF-SN_XHsocket-1-2P-pitch2-5mm_C158012.html" (id 3) (at 193.802 101.854 0)
-      (effects (font (size 1.27 1.27)) hide)
-    )
-    (property "Manufacturer" "JST" (id 4) (at 193.802 104.394 0)
-      (effects (font (size 1.27 1.27)) hide)
-    )
-    (property "LCSC Part" "C158012" (id 5) (at 193.802 106.934 0)
-      (effects (font (size 1.27 1.27)) hide)
-    )
-    (property "JLC Part" "Extended Part" (id 6) (at 193.802 109.474 0)
-      (effects (font (size 1.27 1.27)) hide)
-    )
