File: Hardware/ecu-pcb/vin.kicad_sch (KiCad schematic)
At the start: 10 parts

Commit message: Ecu SCH Ready
Parts:
- removed D?: SMAJ14CA, easyeda2kicad:SMA_L4.3-W2.7-LS5.1-BI, symbol easyeda2kicad:SMAJ14CA_C364287
- removed F?: 33V 750mA Fuse, easyeda2kicad:F1812, symbol easyeda2kicad:33V 750mA Fuse
- added D4: SMAJ14CA, easyeda2kicad:SMA_L4.3-W2.7-LS5.1-BI, symbol easyeda2kicad:SMAJ14CA_C364287
- gave numbers to parts that had none: 8
Connections:
- net GND: now also CN3.1, CN3.3, D4.1
- net at F1.2, Q3.5 (D), Q3.6 (D)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: now also D4.2
Other:
- moved on the sheet: F1

Commit message: PCB Done
Parts:
- added LED3: Red LED 0603, easyeda2kicad:LED0603-R-RD, symbol easyeda2kicad:Red LED 0603
- added R24: 2.2kΩ 0402 50V, easyeda2kicad:R0402, symbol easyeda2kicad:2.2kΩ 0402 50V
- added TP2: TestPoint, TestPoint:TestPoint_Loop_D2.50mm_Drill1.0mm_LowProfile, symbol Connector:TestPoint
Connections:
- net +12V: now also R24.1, TP2.1
- net GND: now also LED3.2 (K)
- new net: LED3.1 (A), R24.2
Changed lines of the file:
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@@
   (junction (at 120.65 61.722) (diameter 0) (color 0 0 0 0)
   )
+  (junction (at 237.998 57.15) (diameter 0) (color 0 0 0 0)
+  )
   (junction (at 202.184 71.882) (diameter 0) (color 0 0 0 0)
   )
@@
     )
     (property "JLC Part" "Basic Part" (id 6) (at 138.43 87.122 0)
+      (effects (font (size 1.27 1.27)) hide)
+    )
+    (pin "1")
+    (pin "2")
+  )
+  (symbol (lib_id "easyeda2kicad:2.2kΩ 0402 50V") (at 237.998 62.23 270) (unit 1)
+    (in_bom yes) (on_board yes) (fields_autoplaced)
+    (property "Reference" "R24" (id 0) (at 240.03 60.9599 90)
+      (effects (font (size 1.27 1.27)) (justify left))
+    )
+    (property "Value" "2.2kΩ 0402 50V" (id 1) (at 240.03 63.4999 90)
+      (effects (font (size 1.27 1.27)) (justify left))
+    )
+    (property "Footprint" "easyeda2kicad:R0402" (id 2) (at 230.378 62.23 0)
+      (effects (font (size 1.27 1.27)) hide)
+    )
+    (property "Datasheet" "https://lcsc.com/product-detail/Chip-Resistor-Surface-Mount-UniOhm_2-2KR-2201-1_C25879.html" (id 3) (at 227.838 62.23 0)
+      (effects (font (size 1.27 1.27)) hide)
+    )
+    (property "Manufacturer" "UNI-ROYAL(厚声)" (id 4) (at 225.298 62.23 0)
+      (effects (font (size 1.27 1.27)) hide)
+    )
+    (property "LCSC Part" "C25879" (id 5) (at 222.758 62.23 0)
+      (effects (font (size 1.27 1.27)) hide)
+    )
+    (property "JLC Part" "Basic Part" (id 6) (at 220.218 62.23 0)
       (effects (font (size 1.27 1.27)) hide)
     )
@@
     )
     (property "Datasheet" "" (id 3) (at 82.296 82.042 0)
+      (effects (font (size 1.27 1.27)) hide)
+    )
+    (pin "1")
+  )
+  (symbol (lib_id "power:+12V") (at 237.998 57.15 270) (unit 1)
+    (in_bom yes) (on_board yes) (fields_autoplaced)
+    (property "Reference" "#PWR0238" (id 0) (at 234.188 57.15 0)
+      (effects (font (size 1.27 1.27)) hide)
+    )
+    (property "Value" "+12V" (id 1) (at 241.3 57.1499 90)
+      (effects (font (size 1.27 1.27)) (justify left))
+    )
+    (property "Footprint" "" (id 2) (at 237.998 57.15 0)
+      (effects (font (size 1.27 1.27)) hide)
+    )
+    (property "Datasheet" "" (id 3) (at 237.998 57.15 0)
+      (effects (font (size 1.27 1.27)) hide)
+    )
+    (pin "1")
+  )
+  (symbol (lib_id "power:GND") (at 237.998 77.47 0) (unit 1)
+    (in_bom yes) (on_board yes) (fields_autoplaced)
+    (property "Reference" "#PWR0237" (id 0) (at 237.998 83.82 0)
+      (effects (font (size 1.27 1.27)) hide)
+    )
+    (property "Value" "GND" (id 1) (at 237.998 82.7532 0))
+    (property "Footprint" "" (id 2) (at 237.998 77.47 0)
+      (effects (font (size 1.27 1.27)) hide)
+    )
+    (property "Datasheet" "" (id 3) (at 237.998 77.47 0)
       (effects (font (size 1.27 1.27)) hide)
     )
@@
     )
     (property "JLC Part" "Extended Part" (id 6) (at 160.782 66.802 0)
+      (effects (font (size 1.27 1.27)) hide)
+    )
+    (pin "1")
+    (pin "2")
+  )
+  (symbol (lib_id "easyeda2kicad:Red LED 0603") (at 239.268 72.39 90) (unit 1)
+    (in_bom yes) (on_board yes) (fields_autoplaced)
+    (property "Reference" "LED3" (id 0) (at 243.586 72.3899 90)
+      (effects (font (size 1.27 1.27)) (justify right))
+    )
+    (property "Value" "Red LED 0603" (id 1) (at 243.586 74.9299 90)
+      (effects (font (size 1.27 1.27)) (justify right))
+    )
+    (property "Footprint" "easyeda2kicad:LED0603-R-RD" (id 2) (at 245.618 72.39 0)
+      (effects (font (size 1.27 1.27)) hide)
+    )
+    (property "Datasheet" "https://lcsc.com/product-detail/Light-Emitting-Diodes-LED_Red-LED-0603_C2286.html" (id 3) (at 248.158 72.39 0)
+      (effects (font (size 1.27 1.27)) hide)
+    )
+    (property "LCSC Part" "C2286" (id 4) (at 250.698 72.39 0)
+      (effects (font (size 1.27 1.27)) hide)
+    )
+    (property "JLC Part" "Basic Part" (id 5) (at 253.238 72.39 0)
       (effects (font (size 1.27 1.27)) hide)
     )
@@
     (pin "8")
   )
+  (symbol (lib_id "Connector:TestPoint") (at 237.998 57.15 90) (unit 1)
+    (in_bom yes) (on_board yes) (fields_autoplaced)
+    (property "Reference" "TP2" (id 0) (at 234.696 50.8 90))
+    (property "Value" "TestPoint" (id 1) (at 234.696 53.34 90))
+    (property "Footprint" "TestPoint:TestPoint_Loop_D2.50mm_Drill1.0mm_LowProfile" (id 2) (at 237.998 52.07 0)
+      (effects (font (size 1.27 1.27)) hide)
+    )
+    (property "Datasheet" "~" (id 3) (at 237.998 52.07 0)
+      (effects (font (size 1.27 1.27)) hide)
+    )
+    (pin "1")
+  )
   (symbol (lib_id "power:+12V") (at 202.184 61.722 0) (unit 1)
