File: Hardware/ecu-pcb/ecu-pcb.kicad_sch (KiCad schematic)
At the start: 8 parts

Commit message: Ecu SCH Ready
Parts:
- added CN1: B2B-XH-A(LF)(SN), easyeda2kicad:CONN-TH_B2B-XH-A-LF-SN, symbol easyeda2kicad:B2B-XH-A(LF)(SN)
- gave numbers to parts that had none: 8
Connections:
- net Audio: now reaches U1.10 (IO25)
- net IO26: now reaches U1.11 (IO26)
- net AMP_ENABLE: now reaches U1.12 (IO27)
- net IO12: now reaches U1.14 (IO12)
- net UART_TX: now reaches U1.27 (IO16)
- net UART_RX: now reaches U1.28 (IO17)
- net APPS2: now reaches U1.4 (SENSOR_VP)
- net APPS1: now reaches U1.5 (SENSOR_VN)
- net IO34: now reaches U1.6 (IO34)
- net IO35: now reaches U1.7 (IO35)
- net IO32: now reaches U1.8 (IO32)
- net IO33: now reaches U1.9 (IO33)
- new net Audio Amp/Speaker+: CN1.2
- new net Audio Amp/Speaker-: CN1.1
Other:
- added sheet 5V Regulator (5V.kicad_sch)
- added sheet APPS (apps.kicad_sch)
- added sheet Audio Amp (PAM8303.kicad_sch)
- added sheet GPIO (gpio.kicad_sch)
- added sheet GPIO1 (gpio.kicad_sch)
- added sheet GPIO2 (gpio.kicad_sch)
- added sheet GPIO3 (gpio.kicad_sch)
- added sheet Sensor Input (sensor.kicad_sch)
- added sheet Sensor Input1 (sensor.kicad_sch)
- added sheet UART (uart.kicad_sch)
- moved on the sheet: R1
